File: hardware/WaterLevel-Eagle-V1/WaterLevel-Eagle-V1.sch (EAGLE design)
At the start: 4 parts, among them IC2 STM8S003F3P6

Commit message: #1 component placement in the PCB
Parts:
- added D1, D3: 1N4148WS-7-F, electroShri:1N4148WS-7-F
- added D2, D4, D5, D6: (no value), electroShri:LED-5MM-REC5MM
- added J1, J2, J3: (no value), electroShri:SCREW-CONN_03-SCREW-5MM
- added K1: RELAY-SPDT, electroShri:RELAY-SPDT
- added PS1: HLK-PM03, electroShri:HLK-PM03
- added Q1, Q2: (no value), eventHorizon:TRANSISTOR_NPNWIDE
- added R1, R5: 10K, eventHorizon:RESISTOR0603
- added R2, R3: (no value), eventHorizon:RESISTOR0805
- added SG1: F/TMB, eventHorizon:F/TMB
Connections:
- new net +5V: D3.K, SG1.+
- new net D0(RX): R5.2
- new net N$1: D1.K, K1.COIL1
- new net N$2: D1.A, K1.COIL2, Q1.C
- new net N$3: Q1.B, R2.1, R3.1
- new net N$4: D3.A, Q2.C, SG1.-
- new net N$5: Q2.B, R1.2, R5.1
- net GND: now also Q1.E, Q2.E, R1.1, R3.2
- net PC5/D7: now also R2.2
Other:
- note added: "Buzzer"
