File: hardware/WaterLevel-STM8-V1/WaterLevel-STM8-V1.brd (EAGLE design)
At the start: 60 x 60 mm, 22 parts, among them IC2 STM8S003F3P6, K1 RELAY-SPDT

Commit message: #1 New PCB update
Parts:
- removed D5, D6: (no value), electroShri:LED_5MM
- removed J1, J2: (no value), electroShri:SCREWTERMINAL-5MM-3
- added A0, SCL, SDA: TPSQTP20R, testpad:TP20R
- added AC_IN, MOTOR, TANK: (no value), electroShri:SCREWTERMINAL-5MM-3
- added C1, C2: 1uF, eventHorizon:C0805
- added FULL, LOW, SYS: (no value), electroShri:LED_5MM
- added GOLD_ORB_SM1: OSHWLOGOLOGO16MM, electroShri:OSHW_16MM
- added J4: (no value), SparkFun-Connectors:1X04
- added J5: (no value), electroShri:6_PIN_SERIAL_TARGET_SIDE_W_SILK
- added R10, R9: 10K, eventHorizon:R0805
- added R6, R7, R8: 330, eventHorizon:R0805
- added VR1: LM1117MPX-3.3, electroShri:VREG_LM1117MPX-3.3
- D2, D4: value (none) -> TPSQTP20R; device electroShri:LED_5MM -> testpad:TP20R
- J3: device electroShri:SCREWTERMINAL-5MM-3 -> electroShri:MOLEX-1X2
- R1, R5: device eventHorizon:R0603 -> eventHorizon:R0805
- R2, R3: value (none) -> 10K
- moved J3 34.0 mm to (3.25, 49.2), turned to 90 degrees
- moved IC2 27.0 mm to (34.0, 39.8), turned to 0 degrees
- moved C8 26.3 mm to (33.8, 34.5), turned to 0 degrees
- moved D1 23.9 mm to (30.5, 30.5), turned to 90 degrees
- moved Q1 23.0 mm to (27.2, 30.8), turned to 270 degrees
- moved R3 22.5 mm to (23.8, 30.8)
- moved R2 22.3 mm to (27.2, 34.2), turned to 0 degrees
- moved SG1 18.6 mm to (66.8, 47.0), turned to 270 degrees
- moved D2 16.9 mm to (23.8, 36.8)
- moved C7 15.9 mm to (28.0, 37.8)
- moved D4 13.1 mm to (23.4, 39.4)
- moved R5 9.65 mm to (51.8, 50.8), turned to 270 degrees
- moved D3 9.41 mm to (59.0, 50.2)
- moved Q2 9.41 mm to (55.5, 50.8)
- moved R4 9.40 mm to (25.8, 42.2), turned to 270 degrees
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Connections:
- removed net D0(RX): R5.2
- new net EARTH: AC_IN.3, MOTOR.3
- new net LIVE: AC_IN.1, K1.1, PS1.1
- new net LIVE-MTR: K1.4, MOTOR.1
- new net N$6: FULL.A, R7.1
- new net N$7: LOW.A, R8.1
- new net NUTRAL: AC_IN.2, MOTOR.2, PS1.2
- net +5V: now also C1.1, D1.1, J3.1, K1.2, PS1.4, VR1.3
- net D13: now also R6.2
- net GND: now also C1.2, C2.2, FULL.K, J3.2, J4.2, J5.P$6, LOW.K, PS1.3, SYS.K, TANK.3, VR1.1
- net N$1: now also R6.1, SYS.A; no longer D1.1, K1.2
- net PA1/D0: now also D4.TP
- net PA3/SS/D2~: now also D2.TP
- net PC3/D5~: now also R5.2
- net PC4/D6~/A0: now also A0.TP
- net PC6/D8~: now also R9.2, TANK.2
- net PC7/D9~: now also R10.2, TANK.1
- net PD2/D11/A1: now also R8.2
- net PD3/D12~/A2: now also R7.2
- net RST: now also J4.1
- net RX: now also J5.P$2
- net SCL: now also SCL.TP
- net SDA: now also SDA.TP
- net SWIM/D10: now also J4.3
- net TX: now also J5.P$3
- net VDD: now also C2.1, J4.4, J5.P$4, R10.1, R9.1, VR1.2, VR1.4
Routing:
- net +5V: track 0.00 -> 134.7 mm, vias 0 -> 1
- net VDD: track 0.00 -> 118.4 mm, vias 0 -> 5
- net NUTRAL: track 0.00 -> 63.3 mm
- net TX: track 0.00 -> 52.3 mm, vias 0 -> 1
- net RX: track 0.00 -> 42.6 mm, vias 0 -> 1
- net RST: track 0.00 -> 42.3 mm, vias 0 -> 1
- net LIVE: track 0.00 -> 35.7 mm
- net N$7: track 0.00 -> 33.0 mm
- net PC3/D5~: track 0.00 -> 29.4 mm, vias 0 -> 2
- net SWIM/D10: track 0.00 -> 26.7 mm, vias 0 -> 1
- net N$1: track 0.00 -> 25.7 mm, vias 0 -> 1
- net N$6: track 0.00 -> 24.8 mm
- net LIVE-MTR: track 0.00 -> 23.5 mm
- net PC6/D8~: track 0.00 -> 20.3 mm
- net PC5/D7: track 0.00 -> 19.8 mm
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- added copper zone on layer 1, net EARTH
- added copper zone on layer 16, net EARTH
Other:
- board size 60 x 60 mm -> 75 x 60 mm
- board text added: "H"
- board text added: "L"
- board text added: "WaterLevel Rev. 2"
- board text added: "https://shridattdudhat.github.io/"
- board text added: "https://shridattdudhat.github.io/Water-Level-Controller_for_Home/"

Commit message: Added I2C connector and  Manual Switch to the board
Parts:
- added J1: (no value), electroShri:MOLEX-1X2
- added J2: (no value), SparkFun-Connectors:1X04
- added JMP1: (no value), PatternAgents-ProtoPads:JMP-3-NO
- moved FULL 2.00 mm to (69.0, 30.0)
- moved D3 1.80 mm to (60.0, 51.8)
- moved Q2 1.80 mm to (56.5, 52.2)
- moved R1 1.80 mm to (56.5, 48.8)
- moved R5 1.80 mm to (52.8, 52.2)
- moved SG1 1.58 mm to (67.2, 48.5)
- moved LOW 1.50 mm to (69.0, 17.5)
- moved AC_IN 0.50 mm to (13.0, 5.00)
- moved K1 0.50 mm to (38.0, 19.0)
- moved MOTOR 0.50 mm to (52.0, 5.00)
- moved PS1 0.50 mm to (11.0, 29.0)
Connections:
- new net N$8: J2.1, JMP1.2
- net +5V: now also JMP1.1
- net GND: now also J1.2, J2.4
- net PC4/D6~/A0: now also J1.1
- net SCL: now also J2.2
- net SDA: now also J2.3
- net VDD: now also JMP1.3
Routing:
- net LIVE: track 35.7 -> 78.5 mm
- net SDA: track 4.74 -> 41.9 mm, vias 0 -> 1
- net +5V: track 134.7 -> 163.4 mm
- net SCL: track 7.67 -> 36.0 mm, vias 0 -> 1
- net VDD: track 118.4 -> 143.3 mm, vias 5 -> 6
- net PC4/D6~/A0: track 4.74 -> 25.8 mm, vias 0 -> 1
- net NUTRAL: track 63.3 -> 67.8 mm
- net N$8: track 0.00 -> 3.16 mm
- net TX: track 52.3 -> 54.6 mm
- net RX: track 42.6 -> 44.3 mm
- net N$7: track 33.0 -> 34.5 mm
- net PC3/D5~: track 29.4 -> 30.3 mm
- net N$2: track 10.2 -> 11.1 mm
- net N$6: track 24.8 -> 25.7 mm
- net GND: track 16.1 -> 15.6 mm
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Other:
- outline, holes or cut-outs redrawn
- board text added: "3V3"
- board text added: "AC-DC"
- board text added: "D5"
- board text added: "D7"
- board text added: "E"
- board text added: "G"
- board text added: "GND"
- board text added: "HIGH-9"
- board text added: "LOW-8"
- board text added: "Made in India [Designed by Shridatt Dudhat] https://shridattdudhat.github.io/"
- board text added: "N"
- board text added: "RST"
- board text added: "SCL"
- board text added: "SDA"
- board text added: "SWIM"
- board text removed: "https://shridattdudhat.github.io/"
